File: LTC3105_Eval/LTC3105_Eval.kicad_sch (KiCad schematic)
At the start: 14 parts, among them J1 Conn_01x05_Pin, J2 Conn_01x05_Pin, U1 LTC3105EMS

Commit message: first draft of layout and schematic
Parts:
- removed JP2: SolderJumper_2_Bridged, Jumper:SolderJumper-2_P1.3mm_Bridged_RoundedPad1.0x1.5mm, symbol Jumper:SolderJumper_2_Bridged
- R1, R2, R3, R4, R5: footprint Resistor_SMD:R_1206_3216Metric -> Resistor_SMD:R_0805_2012Metric
Connections:
- net FB: now also J2.3 (Pin_3), R4.2, R5.1, U1.1 (FB); no longer R2.2, R3.1, U1.3 (FBLDO)
- net GND: now also J1.1 (Pin_1); no longer J1.5 (Pin_5)
- net MPPC: now also J1.2 (Pin_2); no longer J1.4 (Pin_4)
- net POWERGOOD: now also J1.4 (Pin_4); no longer J2.4 (Pin_4)
- net VIN: now also J1.5 (Pin_5); no longer J1.1 (Pin_1)
- net VOUT: now also J2.4 (Pin_4); no longer J2.1 (Pin_1)
- net ~{SHUTDOWN}: now also J1.3 (Pin_3); no longer J2.3 (Pin_3)
- new net FB_LDO: J2.1 (Pin_1), R2.2, R3.1, U1.3 (FBLDO)
Other:
- note added: "TODO:"
- note removed: "TODO: -solve faulty pin7 of LTC3185 symbol"
- moved on the sheet: C1, C2
