File: LTC3105_Eval/LTC3105_Eval.kicad_pcb (KiCad board)
At the start: 2 copper layers, 30.5 x 15.2 mm, 14 parts, among them J1 Conn_01x05_Pin, J2 Conn_01x05_Pin, U1 LTC3105EMS

Commit message: first draft of layout and schematic
Parts:
- removed JP2: SolderJumper_2_Bridged, Jumper:SolderJumper-2_P1.3mm_Bridged_RoundedPad1.0x1.5mm
- added G***: LOGO, ked_symbols:KYD_logo, B.Cu at (138.8, 101.8)
- R1, R2, R3, R4, R5: footprint Resistor_SMD:R_1206_3216Metric -> Resistor_SMD:R_0805_2012Metric
- moved R1 27.2 mm to (131.4, 97.8), turned to 180 degrees
- moved R3 11.7 mm to (148.7, 97.5), turned to 90 degrees
- moved C3 9.26 mm to (131.8, 105.0), turned to 90 degrees
- moved C1 8.62 mm to (145.4, 105.1), turned to -90 degrees
- moved C4 7.57 mm to (141.7, 106.6), turned to -90 degrees
- moved R4 7.51 mm to (140.7, 101.2), turned to 90 degrees
- moved R2 6.85 mm to (145.8, 98.7), turned to 90 degrees
- moved L1 6.48 mm to (136.4, 106.9), turned to 0 degrees
- moved R5 5.93 mm to (143.0, 99.3), turned to 90 degrees
- moved C2 5.93 mm to (148.7, 101.8), turned to -90 degrees
- moved U1 2.71 mm to (137.0, 101.4), turned to -90 degrees
Connections:
- J1 pad 1: VIN -> GND
- J1 pad 2: unconnected-(J1-Pin_2-Pad2) -> MPPC
- J1 pad 3: unconnected-(J1-Pin_3-Pad3) -> ~{SHUTDOWN}
- J1 pad 4: MPPC -> POWERGOOD
- J1 pad 5: GND -> VIN
- J2 pad 1: VOUT -> FB_LDO
- J2 pad 3: ~{SHUTDOWN} -> FB
- J2 pad 4: POWERGOOD -> VOUT
- R2 pad 2: /FB -> FB_LDO
- R3 pad 1: /FB -> FB_LDO
- R4 pad 2: Net-(U1-FB) -> FB
- R5 pad 1: Net-(U1-FB) -> FB
- U1 pad 1: Net-(U1-FB) -> FB
- U1 pad 3: /FB -> FB_LDO
Routing:
- net FB_LDO: track 0.00 -> 19.9 mm
- net LDO_OUT: track 0.00 -> 18.9 mm
- net VOUT: track 0.00 -> 18.8 mm
- net FB: track 0.00 -> 14.8 mm
- net POWERGOOD: track 0.00 -> 14.7 mm
- net VIN: track 0.00 -> 12.7 mm
- net ~{SHUTDOWN}: track 0.00 -> 11.6 mm
- net MPPC: track 0.00 -> 10.9 mm
- net Net-(U1-AUX): track 0.00 -> 4.38 mm
- net /SW: track 0.00 -> 3.99 mm
- net GND: vias 0 -> 9
- added copper zone on B.Cu, net GND
- added copper zone on F.Cu, net GND
Other:
- board size 30.5 x 15.2 mm -> 27.9 x 15.2 mm
- board text added: "FB"
- board text added: "FBL"
- board text added: "GND"
- board text added: "LDO"
- board text added: "LTC3105 EVAL V0.0"
- board text added: "MPC"
- board text added: "OUT"
- board text added: "POK"
- board text added: "VIN"
- board text added: "~{SHD}"

Commit message: small changes to layout
Parts:
- removed G***: LOGO, ked_symbols:KYD_logo
Other:
- board text added: "LTC3105 EVAL V0.0."
- board text added: "© Edwin Koch 2024 licenced under CERN-OHL-P V 2.0"
- board text removed: "LTC3105 EVAL V0.0"

Commit message: added QR code to PCB with the v0 repo branch url
Parts:
- added G***: LOGO, QRCODE.preety:LTC3105_Eval_V0_QRCode_5x5, B.Cu at (133.0, 106.0)

Commit message: work on QR code
Parts:
- moved G*** 5.39 mm to (131.0, 101.0)
Changed lines of the file:
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@@
   )
   (footprint "QRCODE.preety:LTC3105_Eval_V0_QRCode_5x5" (layer "B.Cu")
-    (at 133 106 180)
+    (at 131 101 180)
     (attr board_only exclude_from_pos_files exclude_from_bom)
     (fp_text reference "G***" (at 0 0) (layer "B.SilkS") hide
@@
       (stroke (width 0) (type solid)) (fill solid) (layer "B.SilkS"))
   )
-  (gr_rect (start 145 94.1) (end 148 95.2)
+  (gr_rect (start 144.9 94.4) (end 147.9 95.5)
     (stroke (width 0.2) (type solid)) (fill solid) (layer "F.SilkS"))
   (gr_rect (start 125.73 93.98) (end 153.67 109.22)
@@
     (effects (font (size 0.8 0.8) (thickness 0.12)) (justify left bottom))
   )
-  (gr_text "LTC3105 EVAL V0.0.\n" (at 129.7 95.3) (layer "F.SilkS")
+  (gr_text "LTC3105 EVAL V0.0.\n" (at 129.7 95.6) (layer "F.SilkS")
     (effects (font (size 1 1) (thickness 0.12)) (justify left bottom))
   )

Commit message: work on DRC
Routing:
- net GND: track 0.00 -> 2.20 mm
Other:
- board size 27.9 x 15.2 mm -> 29.1 x 15.2 mm
Changed lines of the file:
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@@
   (gr_rect (start 144.9 94.4) (end 147.9 95.5)
     (stroke (width 0.2) (type solid)) (fill solid) (layer "F.SilkS"))
-  (gr_rect (start 125.73 93.98) (end 153.67 109.22)
+  (gr_rect (start 125.13 93.98) (end 154.27 109.22)
     (stroke (width 0.1) (type default)) (fill none) (layer "Edge.Cuts"))
   (gr_text "© Edwin Koch 2024 \nlicenced under\nCERN-OHL-P V 2.0\n" (at 150.3 103.5) (layer "B.SilkS")
@@
   )
   (dimension (type aligned) (layer "User.1")
-    (pts (xy 125.73 93.98) (xy 153.67 93.98))
+    (pts (xy 125.13 93.98) (xy 154.27 93.98))
     (height -5.08)
-    (gr_text "27.9400 mm" (at 139.7 87.1) (layer "User.1")
+    (gr_text "29.1400 mm" (at 139.7 87.1) (layer "User.1")
       (effects (font (size 1.5 1.5) (thickness 0.3)))
     )
@@
   )
   (dimension (type aligned) (layer "User.1")
-    (pts (xy 125.73 93.98) (xy 125.73 109.22))
+    (pts (xy 125.43 93.98) (xy 125.43 109.22))
     (height 5.08)
-    (gr_text "15.2400 mm" (at 118.85 101.6 90) (layer "User.1")
+    (gr_text "15.2400 mm" (at 118.55 101.6 90) (layer "User.1")
       (effects (font (size 1.5 1.5) (thickness 0.3)))
     )
@@
   )
   (segment (start 150.86 104.14) (end 152.4 104.14) (width 0.5) (layer "F.Cu") (net 1))
-  (segment (start 138.1965 102.1125) (end 140.7 102.1125) (width 0.5) (layer "F.Cu") (net 1))
-  (segment (start 138.192 102.108) (end 138.1965 102.1125) (width 0.5) (layer "F.Cu") (net 1))
-  (segment (start 138.176 102.108) (end 138.192 102.108) (width 0.5) (layer "F.Cu") (net 1))
   (segment (start 145.4 104.75) (end 145.85 105.2) (width 0.5) (layer "F.Cu") (net 1))
-  (segment (start 140.7875 102.2) (end 140.7 102.1125) (width 0.5) (layer "F.Cu") (net 1))
   (segment (start 143.6 102.1) (end 144.1375 102.6375) (width 0.5) (layer "F.Cu") (net 1))
   (segment (start 144.1375 102.6375) (end 145.4 102.6375) (width 0.5) (layer "F.Cu") (net 1))
+  (segment (start 138.1805 102.1125) (end 138.176 102.108) (width 0.5) (layer "F.Cu") (net 1))
   (segment (start 137.975 102.309) (end 137.975 103.55) (width 0.4) (layer "F.Cu") (net 1))
-  (segment (start 140.7125 102.1) (end 143.6 102.1) (width 0.5) (layer "F.Cu") (net 1))
   (segment (start 145.85 105.2) (end 149.8 105.2) (width 0.5) (layer "F.Cu") (net 1))
   (segment (start 138.176 102.108) (end 137.975 102.309) (width 0.4) (layer "F.Cu") (net 1))
   (segment (start 149.8 105.2) (end 150.86 104.14) (width 0.5) (layer "F.Cu") (net 1))
-  (segment (start 140.7 102.1125) (end 140.7125 102.1) (width 0.5) (layer "F.Cu") (net 1))
+  (segment (start 143.6 102.1) (end 140.7125 102.1) (width 0.5) (layer "F.Cu") (net 1))
+  (segment (start 140.7 102.1125) (end 138.1805 102.1125) (width 0.5) (layer "F.Cu") (net 1))
   (segment (start 145.4 102.6375) (end 145.4 104.75) (width 0.5) (layer "F.Cu") (net 1))
+  (segment (start 134.65 99.25) (end 134.6 99.2) (width 0.25) (layer "F.Cu") (net 2))
+  (segment (start 141.6125 98.3875) (end 141.6 98.4) (width 0.25) (layer "F.Cu") (net 2))
+  (segment (start 143 98.3875) (end 141.6125 98.3875) (width 0.25) (layer "F.Cu") (net 2))
+  (segment (start 135.375 99.25) (end 134.65 99.25) (width 0.25) (layer "F.Cu") (net 2))
   (via (at 148.7 106.3) (size 0.8) (drill 0.4) (layers "F.Cu" "B.Cu") (free) (net 2))
   (via (at 133.8 99.2) (size 0.8) (drill 0.4) (layers "F.Cu" "B.Cu") (free) (net 2))
@@
     (polygon
       (pts
-        (xy 125.73 109.22)
-        (xy 125.73 93.98)
-        (xy 153.67 93.98)
-        (xy 153.67 109.22)
+        (xy 125.13 109.22)
+        (xy 125.13 93.98)
+        (xy 154.27 93.98)
+        (xy 154.27 109.22)
       )
     )
